File: pcbs/pcb.kicad_pcb (KiCad board)
At the start: 2 copper layers, 148.3 x 111.7 mm, 39 parts

Commit message: Move a few IO pins around to enable I2C and TRRS communication
Previously the wrong pins were used so TRRS and I2C (for cirque)
wouldn't work. Thanks to (0), I didn't print the previous version of the
board because nothing would work essentially.

(0): https://www.reddit.com/r/ErgoMechKeyboards/comments/13ftrsc/comment/jjwuh69/?utm_source=reddit&utm_medium=web2x&context=3
Parts:
- removed J1: , lib:Jumper
Connections:
- J8 pad 2: B2 -> D0
- J9 pad 2: B3 -> D1
- ROT1 pad 1: O1 -> O4
- S11 pad 1: D4 -> C6
- S12 pad 1: D1 -> D2
- S14 pad 1: C6 -> D7
- S15 pad 1: D2 -> F6
- S8 pad 1: D0 -> D4
- S9 pad 1: D7 -> F7
- TRRS1 pad 3: F6 -> D3
Routing:
- net F7: track 78.4 -> 166.4 mm, vias 1 -> 2
- net D7: track 84.4 -> 18.3 mm
- net D3: track 0.00 -> 34.7 mm
- net O1: track 27.4 -> 0.00 mm
- net D2: track 19.5 -> 44.2 mm
- net F6: track 15.4 -> 39.5 mm, vias 0 -> 1
- net D0: track 59.1 -> 35.3 mm
- net D4: track 37.9 -> 59.7 mm
- net C6: track 17.8 -> 38.5 mm
- net B3: track 33.5 -> 14.9 mm
- net GND: track 899.0 -> 882.1 mm
- net O4: track 10.6 -> 26.1 mm
- net B2: track 26.8 -> 11.6 mm
- net D1: track 45.2 -> 38.6 mm
- net ST: track 22.1 -> 20.7 mm
